File: DamnedBoard/v1.brd (EAGLE design)
At the start: 39 x 16.5 mm, 17 parts, among them U1 EFM32ZG108, U2 MAX44009EDT+T21-0490D-M

Commit message: OSH Parkifying layout.
Parts:
- removed R3: 0, SparkFun-Resistors:0603
- added JP2, JP3: JUMPER-SMT_2_NC_TRACE_NO-SILK, SparkFun-Jumpers:SMT-JUMPER_2_NC_TRACE_NO-SILK
- moved C6 35.6 mm to (12.7, 7.62), turned to 45 degrees
- moved C5 33.0 mm to (11.4, 10.2), turned to 45 degrees
- moved C3 31.4 mm to (21.6, 5.08), turned to 45 degrees
- moved C1 26.4 mm to (11.4, 5.08), turned to 135 degrees
- moved C4 23.0 mm to (21.6, 14.0), turned to 135 degrees
- moved C2 19.4 mm to (24.1, 3.81), turned to 45 degrees
- moved R1 14.6 mm to (47.5, 4.95), turned to 180 degrees
- moved U1 10.9 mm to (14.4, 8.38)
- moved D1 10.1 mm to (46.9, 2.29), turned to 180 degrees
- moved U2 8.03 mm to (11.4, 14.0)
- moved JP1 3.87 mm to (18.0, 2.79), turned to 90 degrees
- moved R2 3.86 mm to (3.30, 4.95)
- moved TC1 2.16 mm to (36.4, 11.9), turned to 270 degrees
- moved D2 2.07 mm to (3.94, 2.29), turned to 0 degrees
- moved G1 1.27 mm to (25.4, 11.4)
Connections:
- removed net N$1: G1.P$1, G1.P$2, G1.P$3, G1.P$4, R3.2
- new net +L: G1.P$1, G1.P$2, JP2.2
- new net +R: G1.P$3, G1.P$4, JP3.2
- net VCC: now also JP2.1, JP3.1; no longer R3.1
Routing:
- net PC1: track 0.00 -> 12.7 mm
- net VCC: track 0.00 -> 12.4 mm
- net N$2: track 0.00 -> 2.67 mm
- added copper zone on layer 1, net +L
- added copper zone on layer 1, net +R
Other:
- board size 39 x 16.5 mm -> 50.8 x 16.5 mm

Commit message: Progress on layout.
Parts:
- removed C3, C4, C5: 0.1uF, SparkFun-Capacitors:0402
- C2, C6: device SparkFun-Capacitors:0603 -> SparkFun-Capacitors:0805
- moved U2 21.1 mm to (29.2, 2.54), turned to 180 degrees
- moved C6 12.3 mm to (23.9, 2.41)
- moved C2 10.5 mm to (14.9, 8.76), turned to 315 degrees
- moved U1 10.2 mm to (23.7, 4.32), turned to 225 degrees
- moved C1 4.58 mm to (15.2, 2.54)
- moved JP1 4.26 mm to (16.8, 6.86), turned to 315 degrees
- moved TC1 3.43 mm to (33.8, 9.78), turned to 180 degrees
Connections:
- net N$5 renamed DCP
- net SWCLK renamed SWCLRIP
- net VCC: no longer C3.2, C4.1, C5.1
- net VSS: no longer C3.1, C4.2, C5.2
Routing:
- net VCC: track 12.4 -> 58.3 mm, vias 0 -> 2
- net PC0: track 0.00 -> 24.9 mm, vias 0 -> 2
- net PC1: track 12.7 -> 34.0 mm
- net NRESET: track 0.00 -> 8.62 mm, vias 0 -> 1
- net SDA: track 0.00 -> 6.23 mm
- net PA0: track 0.00 -> 6.06 mm
- net SCL: track 0.00 -> 6.00 mm
- net N$4: track 0.00 -> 4.09 mm
- net DCP: track 0.00 -> 2.94 mm
- net SWCLRIP: track 0.00 -> 1.99 mm, vias 0 -> 1
- net SWDIO: track 0.00 -> 0.87 mm, vias 0 -> 1
Other:
- outline, holes or cut-outs redrawn

Commit message: Candidate for manufacturing.
Parts:
- removed JP3: JUMPER-SMT_2_NC_TRACE_NO-SILK, SparkFun-Jumpers:SMT-JUMPER_2_NC_TRACE_NO-SILK
- removed TC1: TC2050-IDC, TagConnect:TC2050-IDC
- added J1: CORTEX_DEBUG_SMD, SparkFun-Connectors:SAMTECH_FTSH-105-01
- added TP1, TP2, TP3, TP4: TEST-POINT3, SparkFun-Connectors:PAD.03X.03
- added U$2: (no value), boneyard:32BITS_LOGO
- U$1: value DAMNED -> COPYRIGHT; device boneyard:DAMNED_SILK -> boneyard:COPYRIGHT
- moved U$1 9.63 mm to (10.5, 14.0), flipped to the top
Connections:
- net N$4 renamed AVDD
- removed net SWCLRIP: TC1.4, U1.19
- new net SWDCLK: J1.4, U1.19
- net +R: no longer JP3.2
- net NRESET: now also J1.10; no longer TC1.10
- net SCL: now also TP2.P$1; no longer TC1.8
- net SDA: now also TP1.P$1; no longer TC1.7
- net SWDIO: now also J1.2; no longer TC1.2
- net VCC: now also J1.1; no longer JP3.1, TC1.1
- net VSS: now also J1.3, J1.5, J1.9, TP3.P$1, TP4.P$1; no longer TC1.3, TC1.5, TC1.9
Routing:
- net VCC: track 58.3 -> 98.8 mm, vias 2 -> 5
- net SWDCLK: track 0.00 -> 18.2 mm, vias 0 -> 2
- net SWDIO: track 0.87 -> 17.5 mm, vias 1 -> 2
- net NRESET: track 8.62 -> 22.5 mm, vias 1 -> 2
- net PC1: track 34.0 -> 27.3 mm, vias 0 -> 2
- net N$3: track 0.00 -> 2.67 mm
- net SWCLRIP: track 1.99 -> 0.00 mm, vias 1 -> 0
Other:
- board text added: "32bits.io"
- board text added: "Birds-of-the-Damned!"
- board text added: "SCL"
- board text added: "SDA"
- board text added: "v1.0"
